File: PCB/flypi_pcb_kicad/flypi.sch (KiCad schematic (older format))
At the start: 39 parts, among them CON1 BARREL_JACK, J12 USB_A, P1 PeltS1S2, P10 RGB RG-B, P3 Fan+-, P4 Therm +s-, P5 HP1+-, P6 HP2+-, P7 servo +s-, P8 Ring +-s, P9 I2C +-scsd, Q1 1A_NPN_EBC, Q2 1A-NPN-EBC, Q3 1A_NPN_EBC, Q4 1A_NPN_EBC, U1 LM2596, U2 LM2596, U4 L298N, U5 arduino_mini

Commit message: update PCB, change resistor values: 220 for 270, change resistor footprints (shorter footprint), re-wire npn transistors -> now (-) side is being switched on/off, add some logos, change board license (from CC BY SA to CERN OHL 1.2), update board version 0.7 to 1.0 (as they are not backward compatible anymore)
Parts:
- 1k1, R2, R3, R4, R5: footprint Resistors_THT:R_Box_L13.0mm_W4.0mm_P9.00mm -> Resistor_THT:R_Axial_DIN0411_L9.9mm_D3.6mm_P12.70mm_Horizontal; symbol R -> flypi-rescue:R
- C1, C2, C5, C6: symbol CP1 -> flypi-rescue:CP1
- C10, C7, C8: symbol C -> flypi-rescue:C
- CON1: symbol BARREL_JACK -> flypi-rescue:BARREL_JACK
- D1, D3: symbol D_Schottky -> flypi-rescue:D_Schottky
- J12: symbol USB_A-RESCUE-flypi -> flypi-rescue:USB_A-RESCUE-flypi
- L1, L2: symbol INDUCTOR -> flypi-rescue:INDUCTOR
- P1, P3, P5, P6: symbol Conn_01x02 -> flypi-rescue:Conn_01x02
- P10, P9: symbol Conn_01x04 -> flypi-rescue:Conn_01x04
- P4, P7, P8: symbol Conn_01x03 -> flypi-rescue:Conn_01x03
- Q1, Q2, Q3, Q4: symbol 2N2219 -> flypi-rescue:2N2219
- R1: symbol R -> flypi-rescue:R
- R7, R8, R9: value 220 -> 270; footprint Resistors_THT:R_Box_L13.0mm_W4.0mm_P9.00mm -> Resistor_THT:R_Axial_DIN0411_L9.9mm_D3.6mm_P12.70mm_Horizontal; symbol R -> flypi-rescue:R
- U1, U2: symbol LM2596 -> flypi_components:LM2596
- U4: symbol L298N -> flypi_components:L298N
- U5: symbol arduino_mini -> arduino:arduino_mini
Connections:
- wire segments 176 -> 230
